Commit message: Add explore_lite as submodule

File: install/robot_control_pkg/share/robot_control_pkg/description/ros2_control/diffbot.ros2_control.xacro (robot description, xacro)
@@ -1 +1,30 @@
-/home/dhruvil/argo-test/src/robot_control_pkg/description/ros2_control/diffbot.ros2_control.xacro
+<?xml version="1.0"?>
+<robot xmlns:xacro="http://www.ros.org/wiki/xacro">
+  <xacro:macro name="diffbot_ros2_control" params="name prefix">
+    <ros2_control name="${name}" type="system">
+      <hardware>
+        <plugin>robot_control_pkg/RobotControlHardware</plugin>
+        <param name="left_wheel_name">left_wheel_joint</param>
+        <param name="right_wheel_name">right_wheel_joint</param>
+        <!-- <param name="loop_rate">30</param> -->
+        <param name="device">/dev/ttyUSB0</param>
+        <param name="baud_rate">115200</param>
+        <param name="timeout_ms">50</param>
+        <param name="enc_counts_per_rev">246</param>
+        <param name="pid_p">2.55</param>
+        <param name="pid_i">2.15</param>
+        <param name="pid_d">0.35</param>
+      </hardware>
+      <joint name="${prefix}left_wheel_joint">
+        <command_interface name="velocity"/>
+        <state_interface name="position"/>
+        <state_interface name="velocity"/>
+      </joint>
+      <joint name="${prefix}right_wheel_joint">
+        <command_interface name="velocity"/>
+        <state_interface name="position"/>
+        <state_interface name="velocity"/>
+      </joint>
+    </ros2_control>
+  </xacro:macro>
+</robot>

File: install/robot_control_pkg/share/robot_control_pkg/description/urdf/diffbot.urdf.xacro (robot description, xacro)
@@ -1 +1,12 @@
-/home/dhruvil/argo-test/src/robot_control_pkg/description/urdf/diffbot.urdf.xacro
+<?xml version="1.0"?>
+<!-- Basic differential drive mobile base -->
+<robot xmlns:xacro="http://www.ros.org/wiki/xacro" name="diffbot">
+  <xacro:arg name="prefix" default="" />
+  <!-- Import robot's main urdf file -->
+  <xacro:include filename="$(find robot_control_pkg)/urdf/diffbot_description.urdf.xacro" />
+  <!-- Import diffbot ros2_control description -->
+  <xacro:include filename="$(find robot_control_pkg)/ros2_control/diffbot.ros2_control.xacro" />
+  <xacro:diffbot prefix="$(arg prefix)" />
+  <xacro:diffbot_ros2_control
+    name="diffbot" prefix="$(arg prefix)" />
+</robot>

File: install/robot_control_pkg/share/robot_control_pkg/description/urdf/diffbot_description.urdf.xacro (robot description, xacro)
@@ -1 +1,340 @@
-/home/dhruvil/argo-test/src/robot_control_pkg/description/urdf/diffbot_description.urdf.xacro
+<?xml version="1.0" ?>
+<robot xmlns:xacro="http://ros.org/wiki/xacro">
+<xacro:macro name="diffbot" params="prefix">
+<link name="base_link">
+</link>
+<link name="base_footprint_link">
+</link>
+<joint name="base_footprint_joint" type="fixed">
+  <parent link="base_link"/>
+  <child link="base_footprint_link"/>
+  <origin xyz="0 0 0" rpy="0 0 0"/>
+</joint>
+<link
+    name="chassis_link">
+    <inertial>
+      <origin
+        xyz="0.0016049 7.4296E-14 0.058697"
+        rpy="0 0 0" />
+      <mass
+        value="12" />
+      <inertia
+        ixx="0.37085"
+        ixy="5.9421E-08"
+        ixz="-0.0043358"
+        iyy="0.56013"
+        iyz="1.0073E-08"
+        izz="0.86077" />
+    </inertial>
+    <visual>
+      <origin
+        xyz="0 0 0"
+        rpy="0 0 0" />
+      <geometry>
+        <mesh
+          filename="package://robot_control_pkg/description/models/base_link.STL" />
+      </geometry>
+      <material
+        name="">
+        <color
+          rgba="0.29804 0.29804 0.29804 1" />
+      </material>
+    </visual>
+    <collision>
+      <origin
+        xyz="0 0 0"
+        rpy="0 0 0" />
+      <geometry>
+        <mesh
+          filename="package://robot_control_pkg/description/models/base_link.STL" />
+      </geometry>
+    </collision>
+  </link>
+  <joint name="chassis_joint" type="fixed">
+    <parent link="base_link"/>
+    <child link="chassis_link"/>
+    <origin xyz="0 0 0"/>
+  </joint>
+  <link
+    name="right_wheel_link">
+    <inertial>
+      <origin
+        xyz="1.3878E-17 0 -0.0033337"
+        rpy="0 0 0" />
+      <mass
+        value="0.60765" />
+      <inertia
+        ixx="0.0012132"
+        ixy="-1.1019E-20"
+        ixz="5.4221E-19"
+        iyy="0.0012132"
+        iyz="-7.6446E-20"
+        izz="0.0022643" />
+    </inertial>
+    <visual>
+      <origin
+        xyz="0 0 0"
+        rpy="0 0 0" />
+      <geometry>
+        <mesh
+          filename="package://robot_control_pkg/description/models/right_wheel_link.STL" />
+      </geometry>
+      <material
+        name="">
+        <color
+          rgba="0.29804 0.29804 0.29804 1" />
+      </material>
+    </visual>
+    <collision>
+      <origin
+        xyz="0 0 0"
+        rpy="0 0 0" />
+      <geometry>
+        <mesh
+          filename="package://robot_control_pkg/description/models/right_wheel_link.STL" />
+      </geometry>
+    </collision>
+  </link>
+  <joint
+    name="right_wheel_joint"
+    type="continuous">
+    <origin
+      xyz="0 -0.21525 0.059"
+      rpy="1.5708 0 0" />
+    <parent
+      link="chassis_link" />
+    <child
+      link="right_wheel_link" />
+    <axis
+      xyz="0 0 -1" />
+    <limit
+      effort="10"
+      velocity="10" />
+    <dynamics
+      damping="0.1"
+      friction="0.1" />
+  </joint>
+  <link
+    name="left_wheel_link">
+    <inertial>
+      <origin
+        xyz="6.9389E-18 0 -0.0033337"
+        rpy="0 0 0" />
+      <mass
+        value="0.60765" />
+      <inertia
+        ixx="0.0012132"
+        ixy="2.0023E-20"
+        ixz="1.2266E-19"
+        iyy="0.0012132"
+        iyz="1.6778E-19"
+        izz="0.0022643" />
+    </inertial>
+    <visual>
+      <origin
+        xyz="0 0 0"
+        rpy="0 0 0" />
+      <geometry>
+        <mesh
+          filename="package://robot_control_pkg/description/models/left_wheel_link.STL" />
+      </geometry>
+      <material
+        name="">
+        <color
+          rgba="0.29804 0.29804 0.29804 1" />
+      </material>
+    </visual>
+    <collision>
+      <origin
+        xyz="0 0 0"
+        rpy="0 0 0" />
+      <geometry>
+        <mesh
+          filename="package://robot_control_pkg/description/models/left_wheel_link.STL" />
+      </geometry>
+    </collision>
+  </link>
+  <joint
+    name="left_wheel_joint"
+    type="continuous">
+    <origin
+      xyz="0 0.21525 0.059"
+      rpy="-1.5708 0 0" />
+    <parent
+      link="chassis_link" />
+    <child
+      link="left_wheel_link" />
+    <axis
+      xyz="0 0 1" />
+    <limit
+      effort="10"
+      velocity="10" />
+    <dynamics
+      damping="0.1"
+      friction="0.1" />
+  </joint>
+  <link
+    name="front_caster_link">
+    <inertial>
+      <origin
+        xyz="-1.7347E-18 0.0030758 -0.00021456"
+        rpy="0 0 0" />
+      <mass
+        value="0.05" />
+      <inertia
+        ixx="3.1756E-06"
+        ixy="-4.0907E-23"
+        ixz="-7.1759E-22"
+        iyy="6.1712E-06"
+        iyz="-5.9858E-09"
+        izz="3.1557E-06" />
+    </inertial>
+    <visual>
+      <origin
+        xyz="0 0 0"
+        rpy="0 0 0" />
+      <geometry>
+        <mesh
+          filename="package://robot_control_pkg/description/models/front_caster_link.STL" />
+      </geometry>
+      <material
+        name="">
+        <color
+          rgba="0.75294 0.75294 0.75294 1" />
+      </material>
+    </visual>
+    <collision>
+      <origin
+        xyz="0 0 0"
+        rpy="0 0 0" />
+      <geometry>
+        <mesh
+          filename="package://robot_control_pkg/description/models/front_caster_link.STL" />
+      </geometry>
+    </collision>
+  </link>
+  <joint
+    name="front_caster_joint"
+    type="fixed">
+    <origin
+      xyz="0.24008 0 -0.0075"
+      rpy="1.5708 0 1.5708" />
+    <parent
+      link="chassis_link" />
+    <child
+      link="front_caster_link" />
+    <axis
+      xyz="0 0 0" />
+    <dynamics
+      damping="0"
+      friction="0.001" />
+  </joint>
+  <link
+    name="rear_caster_link">
+    <inertial>
+      <origin
+        xyz="-3.2526E-19 0.0030758 -0.00021456"
+        rpy="0 0 0" />
+      <mass
+        value="0.05" />
+      <inertia
+        ixx="3.1756E-06"
+        ixy="-5.5022E-23"
+        ixz="-1.1135E-21"
+        iyy="6.1712E-06"
+        iyz="-5.9858E-09"
+        izz="3.1557E-06" />
+    </inertial>
+    <visual>
+      <origin
+        xyz="0 0 0"
+        rpy="0 0 0" />
+      <geometry>
+        <mesh
+          filename="package://robot_control_pkg/description/models/rear_caster_link.STL" />
+      </geometry>
+      <material
+        name="">
+        <color
+          rgba="0.75294 0.75294 0.75294 1" />
+      </material>
+    </visual>
+    <collision>
+      <origin
+        xyz="0 0 0"
+        rpy="0 0 0" />
+      <geometry>
+        <mesh
+          filename="package://robot_control_pkg/description/models/rear_caster_link.STL" />
+      </geometry>
+    </collision>
+  </link>
+  <joint
+    name="rear_caster_joint"
+    type="fixed">
+    <origin
+      xyz="-0.23992 0 -0.0075"
+      rpy="1.5708 0 1.5708" />
+    <parent
+      link="chassis_link" />
+    <child
+      link="rear_caster_link" />
+    <axis
+      xyz="0 0 0" />
+    <dynamics
+      damping="0"
+      friction="0.001" />
+  </joint>
+  <link
+    name="lidar_link">
+    <inertial>
+      <origin
+        xyz="2.7756E-17 -1.0842E-19 0.0045392"
+        rpy="0 0 0" />
+      <mass
+        value="0.25" />
+      <inertia
+        ixx="4.9112E-05"
+        ixy="0"
+        ixz="-1.2331E-21"
+        iyy="4.9112E-05"
+        iyz="-4.2562E-37"
+        izz="8.3852E-05" />
+    </inertial>
+    <visual>
+      <origin
+        xyz="0 0 0"
+        rpy="0 0 0" />
+      <geometry>
+        <mesh
+          filename="package://robot_control_pkg/description/models/lidar_link.STL" />
+      </geometry>
+      <material
+        name="">
+        <color
+          rgba="0.10196 0.10196 0.10196 1" />
+      </material>
+    </visual>
+    <collision>
+      <origin
+        xyz="0 0 0"
+        rpy="0 0 0" />
+      <geometry>
+        <mesh
+          filename="package://robot_control_pkg/description/models/lidar_link.STL" />
+      </geometry>
+    </collision>
+  </link>
+  <joint
+    name="lidar_joint"
+    type="fixed">
+    <origin
+      xyz="0.19 0 0.24025"
+      rpy="0 0 3.14159" />
+    <parent
+      link="chassis_link" />
+    <child
+      link="lidar_link" />
+  </joint>
+  </xacro:macro>
+</robot>

File: install/simulation_pkg/share/simulation_pkg/description/gazebo_control.xacro (robot description, xacro)
@@ -1 +1,28 @@
-/home/dhruvil/argo-test/build/simulation_pkg/description/gazebo_control.xacro
+<?xml version="1.0"?>
+<robot xmlns:xacro="http://ros.org/wiki/xacro">
+    <gazebo>
+        <plugin filename="gz-sim-diff-drive-system" name="gz::sim::systems::DiffDrive">
+            <!-- Remove <ros> tag. -->
+            <!-- wheels -->
+            <left_joint>left_wheel_joint</left_joint>
+            <right_joint>right_wheel_joint</right_joint>
+            <!-- kinematics -->
+            <wheel_separation>0.385</wheel_separation>
+            <wheel_radius>0.08</wheel_radius> <!-- computed from <wheel_diameter> in the original plugin-->
+            <!-- limits -->
+            <max_linear_acceleration>10</max_linear_acceleration> <!-- computed from <max_linear_acceleration> in the original plugin-->
+            <topic>cmd_vel</topic> <!-- from <commant_topic> -->
+            <odom_topic>odom</odom_topic> <!-- from <odometry_topic> -->
+            <frame_id>odom</frame_id> <!-- from <odometry_frame> -->
+            <child_frame_id>base_link</child_frame_id> <!-- from <robot_base_frame> -->
+            <odom_publisher_frequency>30</odom_publisher_frequency> <!-- from <update_rate>-->
+            <tf_topic>/tf</tf_topic> <!-- Short topic name for tf output -->
+        </plugin>
+        <plugin filename="gz-sim-joint-state-publisher-system"
+            name="gz::sim::systems::JointStatePublisher">
+            <topic>joint_states</topic> <!--from <ros><remapping> -->
+            <joint_name>left_wheel_joint</joint_name>
+            <joint_name>right_wheel_joint</joint_name>
+        </plugin>
+    </gazebo>
+</robot>

File: install/simulation_pkg/share/simulation_pkg/description/gazebo_references.xacro (robot description, xacro)
@@ -1 +1,18 @@
-/home/dhruvil/argo-test/build/simulation_pkg/description/gazebo_references.xacro
+<?xml version="1.0"?>
+<robot xmlns:xacro="http://ros.org/wiki/xacro">
+    <gazebo reference="chassis_link">
+        <material>Gazebo/White</material>
+    </gazebo>
+    <gazebo reference="right_wheel_link">
+        <material>Gazebo/Black</material>
+    </gazebo>
+    <gazebo reference="left_wheel_link">
+        <material>Gazebo/Black</material>
+    </gazebo>
+    <gazebo reference="front_caster_link">
+        <material>Gazebo/Grey</material>
+    </gazebo>
+    <gazebo reference="rear_caster_link">
+        <material>Gazebo/Grey</material>
+    </gazebo>
+</robot>

File: install/simulation_pkg/share/simulation_pkg/description/lidar.xacro (robot description, xacro)
@@ -1 +1,35 @@
-/home/dhruvil/argo-test/build/simulation_pkg/description/lidar.xacro
+<?xml version="1.0"?>
+<robot xmlns:xacro="http://ros.org/wiki/xacro">
+    <gazebo reference="lidar_link">
+        <material>Gazebo/Black</material>
+        <sensor name='gpu_lidar' type='gpu_lidar'>
+            <always_on>true</always_on>
+            <visualize>true</visualize>
+            <pose>0 0 0 0 0 0</pose>
+            <update_rate>5</update_rate>
+            <topic>scan</topic>
+            <gz_frame_id>lidar_link</gz_frame_id>
+            <lidar>
+                <scan>
+                    <horizontal>
+                        <samples>640</samples>
+                        <resolution>1</resolution>
+                        <min_angle>-3.1416</min_angle>
+                        <max_angle>3.1416</max_angle>
+                    </horizontal>
+                    <vertical>
+                        <samples>1</samples>
+                        <resolution>0.01</resolution>
+                        <min_angle>0</min_angle>
+                        <max_angle>0</max_angle>
+                    </vertical>
+                </scan>
+                <range>
+                    <min>0.5</min>
+                    <max>8.0</max>
+                    <resolution>0.01</resolution>
+                </range>
+            </lidar>
+        </sensor>
+    </gazebo>
+</robot>

File: install/simulation_pkg/share/simulation_pkg/description/robot_core.xacro (robot description, xacro)
@@ -1 +1,336 @@
-/home/dhruvil/argo-test/build/simulation_pkg/description/robot_core.xacro
+<?xml version="1.0" ?>
+<robot xmlns:xacro="http://ros.org/wiki/xacro">
+<link name="base_link">
+</link>
+<link name="base_footprint_link">
+</link>
+<joint name="base_footprint_joint" type="fixed">
+  <parent link="base_link"/>
+  <child link="base_footprint_link"/>
+  <origin xyz="0 0 0" rpy="0 0 0"/>
+</joint>
+<link
+    name="chassis_link">
+    <inertial>
+      <origin
+        xyz="0.0016049 7.4296E-14 0.058697"
+        rpy="0 0 0" />
+      <mass
+        value="12" />
+      <inertia
+        ixx="0.37085"
+        ixy="5.9421E-08"
+        ixz="-0.0043358"
+        iyy="0.56013"
+        iyz="1.0073E-08"
+        izz="0.86077" />
+    </inertial>
+    <visual>
+      <origin
+        xyz="0 0 0"
+        rpy="0 0 0" />
+      <geometry>
+        <mesh
+          filename="package://simulation_pkg/models/base_link.STL" />
+      </geometry>
+      <material
+        name="">
+        <color
+          rgba="0.29804 0.29804 0.29804 1" />
+      </material>
+    </visual>
+    <collision>
+      <origin
+        xyz="0 0 0"
+        rpy="0 0 0" />
+      <geometry>
+        <mesh
+          filename="package://simulation_pkg/models/base_link.STL" />
+      </geometry>
+    </collision>
+  </link>
+  <joint name="chassis_joint" type="fixed">
+    <parent link="base_link"/>
+    <child link="chassis_link"/>
+    <origin xyz="0 0 0"/>
+  </joint>
+  <link
+    name="right_wheel_link">
+    <inertial>
+      <origin
+        xyz="1.3878E-17 0 -0.0033337"
+        rpy="0 0 0" />
+      <mass
+        value="0.60765" />
+      <inertia
+        ixx="0.0012132"
+        ixy="-1.1019E-20"
+        ixz="5.4221E-19"
+        iyy="0.0012132"
+        iyz="-7.6446E-20"
+        izz="0.0022643" />
+    </inertial>
+    <visual>
+      <origin
+        xyz="0 0 0"
+        rpy="0 0 0" />
+      <geometry>
+        <mesh
+          filename="package://simulation_pkg/models/right_wheel_link.STL" />
+      </geometry>
+      <material
+        name="">
+        <color
+          rgba="0.29804 0.29804 0.29804 1" />
+      </material>
+    </visual>
+    <collision>
+      <origin
+        xyz="0 0 0"
+        rpy="0 0 0" />
+      <geometry>
+        <sphere radius="0.08"/>
+      </geometry>
+    </collision>
+  </link>
+  <joint
+    name="right_wheel_joint"
+    type="continuous">
+    <origin
+      xyz="0 -0.21525 0.059"
+      rpy="1.5708 0 0" />
+    <parent
+      link="chassis_link" />
+    <child
+      link="right_wheel_link" />
+    <axis
+      xyz="0 0 -1" />
+    <limit
+      effort="10"
+      velocity="10" />
+    <dynamics
+      damping="0.1"
+      friction="0.1" />
+  </joint>
+  <link
+    name="left_wheel_link">
+    <inertial>
+      <origin
+        xyz="6.9389E-18 0 -0.0033337"
+        rpy="0 0 0" />
+      <mass
+        value="0.60765" />
+      <inertia
+        ixx="0.0012132"
+        ixy="2.0023E-20"
+        ixz="1.2266E-19"
+        iyy="0.0012132"
+        iyz="1.6778E-19"
+        izz="0.0022643" />
+    </inertial>
+    <visual>
+      <origin
+        xyz="0 0 0"
+        rpy="0 0 0" />
+      <geometry>
+        <mesh
+          filename="package://simulation_pkg/models/left_wheel_link.STL" />
+      </geometry>
+      <material
+        name="">
+        <color
+          rgba="0.29804 0.29804 0.29804 1" />
+      </material>
+    </visual>
+    <collision>
+      <origin
+        xyz="0 0 0"
+        rpy="0 0 0" />
+      <geometry>
+        <sphere radius="0.08"/>
+      </geometry>
+    </collision>
+  </link>
+  <joint
+    name="left_wheel_joint"
+    type="continuous">
+    <origin
+      xyz="0 0.21525 0.059"
+      rpy="-1.5708 0 0" />
+    <parent
+      link="chassis_link" />
+    <child
+      link="left_wheel_link" />
+    <axis
+      xyz="0 0 1" />
+    <limit
+      effort="10"
+      velocity="10" />
+    <dynamics
+      damping="0.1"
+      friction="0.1" />
+  </joint>
+  <link
+    name="front_caster_link">
+    <inertial>
+      <origin
+        xyz="-1.7347E-18 0.0030758 -0.00021456"
+        rpy="0 0 0" />
+      <mass
+        value="0.05" />
+      <inertia
+        ixx="3.1756E-06"
+        ixy="-4.0907E-23"
+        ixz="-7.1759E-22"
+        iyy="6.1712E-06"
+        iyz="-5.9858E-09"
+        izz="3.1557E-06" />
+    </inertial>
+    <visual>
+      <origin
+        xyz="0 0 0"
+        rpy="0 0 0" />
+      <geometry>
+        <mesh
+          filename="package://simulation_pkg/models/front_caster_link.STL" />
+      </geometry>
+      <material
+        name="">
+        <color
+          rgba="0.75294 0.75294 0.75294 1" />
+      </material>
+    </visual>
+    <collision>
+      <origin
+        xyz="0 0 0"
+        rpy="0 0 0" />
+      <geometry>
+        <mesh
+          filename="package://simulation_pkg/models/front_caster_link.STL" />
+      </geometry>
+    </collision>
+  </link>
+  <joint
+    name="front_caster_joint"
+    type="fixed">
+    <origin
+      xyz="0.24008 0 -0.0075"
+      rpy="1.5708 0 1.5708" />
+    <parent
+      link="chassis_link" />
+    <child
+      link="front_caster_link" />
+    <axis
+      xyz="0 0 0" />
+    <dynamics
+      damping="0"
+      friction="0.001" />
+  </joint>
+  <link
+    name="rear_caster_link">
+    <inertial>
+      <origin
+        xyz="-3.2526E-19 0.0030758 -0.00021456"
+        rpy="0 0 0" />
+      <mass
+        value="0.05" />
+      <inertia
+        ixx="3.1756E-06"
+        ixy="-5.5022E-23"
+        ixz="-1.1135E-21"
+        iyy="6.1712E-06"
+        iyz="-5.9858E-09"
+        izz="3.1557E-06" />
+    </inertial>
+    <visual>
+      <origin
+        xyz="0 0 0"
+        rpy="0 0 0" />
+      <geometry>
+        <mesh
+          filename="package://simulation_pkg/models/rear_caster_link.STL" />
+      </geometry>
+      <material
+        name="">
+        <color
+          rgba="0.75294 0.75294 0.75294 1" />
+      </material>
+    </visual>
+    <collision>
+      <origin
+        xyz="0 0 0"
+        rpy="0 0 0" />
+      <geometry>
+        <mesh
+          filename="package://simulation_pkg/models/rear_caster_link.STL" />
+      </geometry>
+    </collision>
+  </link>
+  <joint
+    name="rear_caster_joint"
+    type="fixed">
+    <origin
+      xyz="-0.23992 0 -0.0075"
+      rpy="1.5708 0 1.5708" />
+    <parent
+      link="chassis_link" />
+    <child
+      link="rear_caster_link" />
+    <axis
+      xyz="0 0 0" />
+    <dynamics
+      damping="0"
+      friction="0.001" />
+  </joint>
+  <link
+    name="lidar_link">
+    <inertial>
+      <origin
+        xyz="2.7756E-17 -1.0842E-19 0.0045392"
+        rpy="0 0 0" />
+      <mass
+        value="0.25" />
+      <inertia
+        ixx="4.9112E-05"
+        ixy="0"
+        ixz="-1.2331E-21"
+        iyy="4.9112E-05"
+        iyz="-4.2562E-37"
+        izz="8.3852E-05" />
+    </inertial>
+    <visual>
+      <origin
+        xyz="0 0 0"
+        rpy="0 0 0" />
+      <geometry>
+        <mesh
+          filename="package://simulation_pkg/models/lidar_link.STL" />
+      </geometry>
+      <material
+        name="">
+        <color
+          rgba="0.10196 0.10196 0.10196 1" />
+      </material>
+    </visual>
+    <collision>
+      <origin
+        xyz="0 0 0"
+        rpy="0 0 0" />
+      <geometry>
+        <mesh
+          filename="package://simulation_pkg/models/lidar_link.STL" />
+      </geometry>
+    </collision>
+  </link>
+  <joint
+    name="lidar_joint"
+    type="fixed">
+    <origin
+      xyz="0.19 0 0.24025"
+      rpy="0 0 0" />
+    <parent
+      link="chassis_link" />
+    <child
+      link="lidar_link" />
+  </joint>
+</robot>

File: install/simulation_pkg/share/simulation_pkg/description/robot_urdf.xacro (robot description, xacro)
@@ -1 +1,8 @@
-/home/dhruvil/argo-test/build/simulation_pkg/description/robot_urdf.xacro
+<?xml version="1.0"?>
+<robot name="sim_robot" xmlns:xacro="http://ros.org/wiki/xacro">
+    <xacro:include filename="robot_core.xacro" />
+    <!-- <xacro:include filename="gazebo_control.xacro" /> -->
+    <xacro:include filename="ros2_control.xacro" />
+    <xacro:include filename="gazebo_references.xacro" />
+    <xacro:include filename="lidar.xacro" />
+</robot>
